File: hw/sch_pcb/OPTMAGPROBE01A.kicad_pcb (KiCad board)
At the start: 2 copper layers, 6 parts, among them J1 HEADER_1x03, U1 AH3572, U2 VCNT2020

Commit message: Edit
Parts:
- added M3: HOLE, Mlab_Mechanical:dira_3mm, F.Cu at (8.89, -10.0)
- added M4: HOLE, Mlab_Mechanical:dira_3mm, F.Cu at (15.2, -11.6)
- J1: footprint Mlab_Pin_Headers:Angled_1x03 -> Mlab_Pin_Headers:Straight_1x03; moved to B.Cu
- R2, U2: moved to B.Cu
- moved U1 143.8 mm to (12.0, -3.05)
- moved U2 143.4 mm to (12.0, -7.05)
- moved R2 142.2 mm to (6.86, -6.86), turned to 90 degrees
- moved R1 138.2 mm to (8.89, -5.05), turned to -90 degrees
- moved C1 135.2 mm to (6.99, -3.02), turned to -90 degrees
- moved J1 134.3 mm to (4.07, -5.00), turned to 180 degrees
Other:
- board outline added: 14 x 10 mm

Commit message: Edit
Parts:
- moved M4 13.1 mm to (9.00, 0.00)
Routing:
- net /COUNT: track 0.00 -> 17.0 mm, vias 0 -> 2
- net +5V: track 0.00 -> 13.3 mm, vias 0 -> 2
- net GND: track 0.00 -> 12.8 mm, vias 0 -> 6
- net Net-(R1-Pad2): track 0.00 -> 5.14 mm
- added copper zone on B.Cu, net GND
- added copper zone on F.Cu, net GND
Other:
- board text added: "+5V"
- board text added: "GND"
- board text added: "OUT"
- board text added: "TFPROBE01A"
- board text added: "ThunderFly"
