File: hw/sch_pcb/OPTMAGPROBE01A.kicad_sch (KiCad schematic)
At the start: 6 parts, among them J1 HEADER_1x03, U1 AH3572, U2 VCNT2020

Commit message: Edit
Parts:
- added M3, M4: HOLE, Mlab_Mechanical:dira_3mm, symbol MLAB_MECHANICAL:HOLE
- J1: footprint Mlab_Pin_Headers:Angled_1x03 -> Mlab_Pin_Headers:Straight_1x03
Connections:
- no-connect marks 0 -> 2
Changed lines of the file:
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@@
   (junction (at 146.05 109.22) (diameter 1.016) (color 0 0 0 0))
   (junction (at 156.21 111.76) (diameter 1.016) (color 0 0 0 0))
+  (no_connect (at 257.81 17.78))
+  (no_connect (at 266.7 17.78))
   (wire (pts (xy 71.12 96.52) (xy 71.12 97.79))
     (stroke (width 0) (type solid) (color 0 0 0 0))
@@
     (effects (font (size 1.27 1.27)) (justify right bottom))
   )
+  (symbol (lib_id "MLAB_MECHANICAL:HOLE") (at 257.81 16.51 270) (unit 1)
+    (in_bom yes) (on_board yes)
+    (property "Reference" "M3" (id 0) (at 259.2071 15.6007 90)
+      (effects (font (size 1.524 1.524)) (justify left))
+    )
+    (property "Value" "HOLE" (id 1) (at 259.2071 18.3083 90)
+      (effects (font (size 1.524 1.524)) (justify left))
+    )
+    (property "Footprint" "Mlab_Mechanical:dira_3mm" (id 2) (at 257.81 16.51 0)
+      (effects (font (size 1.524 1.524)) hide)
+    )
+    (property "Datasheet" "" (id 3) (at 257.81 16.51 0)
+      (effects (font (size 1.524 1.524)))
+    )
+  )
+  (symbol (lib_id "MLAB_MECHANICAL:HOLE") (at 266.7 16.51 270) (unit 1)
+    (in_bom yes) (on_board yes)
+    (property "Reference" "M4" (id 0) (at 268.0971 15.6007 90)
+      (effects (font (size 1.524 1.524)) (justify left))
+    )
+    (property "Value" "HOLE" (id 1) (at 268.0971 18.3083 90)
+      (effects (font (size 1.524 1.524)) (justify left))
+    )
+    (property "Footprint" "Mlab_Mechanical:dira_3mm" (id 2) (at 266.7 16.51 0)
+      (effects (font (size 1.524 1.524)) hide)
+    )
+    (property "Datasheet" "" (id 3) (at 266.7 16.51 0)
+      (effects (font (size 1.524 1.524)))
+    )
+  )
   (symbol (lib_id "power:+5V") (at 71.12 96.52 0) (unit 1)
     (in_bom yes) (on_board yes)
@@
       (effects (font (size 1.524 1.524)) (justify left) hide)
     )
-    (property "Footprint" "Mlab_Pin_Headers:Angled_1x03" (id 2) (at 163.83 109.22 0)
+    (property "Footprint" "Mlab_Pin_Headers:Straight_1x03" (id 2) (at 163.83 109.22 0)
       (effects (font (size 1.524 1.524)) hide)
     )
@@
     )
     (path "/d81e7dca-ab0d-4e13-984a-1c5b00f3383c"
-      (reference "J1") (unit 1) (value "HEADER_1x03") (footprint "Mlab_Pin_Headers:Angled_1x03")
+      (reference "J1") (unit 1) (value "HEADER_1x03") (footprint "Mlab_Pin_Headers:Straight_1x03")
+    )
+    (path "/196227d8-be2a-4b6f-852b-6ff909ae9882"
+      (reference "M3") (unit 1) (value "HOLE") (footprint "Mlab_Mechanical:dira_3mm")
+    )
+    (path "/3b547b03-2d6f-403a-a314-16fe37d96cd6"
+      (reference "M4") (unit 1) (value "HOLE") (footprint "Mlab_Mechanical:dira_3mm")
     )
     (path "/9e12790b-cec9-4dd8-a3af-c20d5c11d549"

Commit message: Edit bom
Parts:
- C1: UST_ID (none) -> 5c70984812875079b91f8bf2
- R1: UST_ID (none) -> 5c70984512875079b91f8957
- U1: UST_ID (none) -> 5f9d011812875025b39777ea
- U2: UST_ID (none) -> 5f9d106a12875025b39777fa
Changed lines of the file:
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@@
   (junction (at 146.05 109.22) (diameter 1.016) (color 0 0 0 0))
   (junction (at 156.21 111.76) (diameter 1.016) (color 0 0 0 0))
+  (no_connect (at 266.7 17.78))
   (no_connect (at 257.81 17.78))
-  (no_connect (at 266.7 17.78))
   (wire (pts (xy 71.12 96.52) (xy 71.12 97.79))
     (stroke (width 0) (type solid) (color 0 0 0 0))
@@
       (effects (font (size 1.27 1.27)) hide)
     )
+    (property "UST_ID" "5c70984512875079b91f8957" (id 4) (at 71.12 101.6 0)
+      (effects (font (size 1.27 1.27)) hide)
+    )
   )
   (symbol (lib_id "Device:R") (at 146.05 102.87 0) (unit 1)
@@
     )
     (property "Datasheet" "~" (id 3) (at 146.05 116.84 0)
+      (effects (font (size 1.27 1.27)) hide)
+    )
+    (property "UST_ID" "5c70984812875079b91f8bf2" (id 4) (at 146.05 116.84 0)
       (effects (font (size 1.27 1.27)) hide)
     )
@@
     )
     (property "Datasheet" "https://cz.mouser.com/datasheet/2/115/AH3572-1483253.pdf" (id 3) (at 90.17 64.77 0)
+      (effects (font (size 1.27 1.27)) hide)
+    )
+    (property "UST_ID" "5f9d011812875025b39777ea" (id 4) (at 90.17 64.77 0)
       (effects (font (size 1.27 1.27)) hide)
     )
@@
       (effects (font (size 1.27 1.27)) (justify left bottom) hide)
     )
-  )
+    (property "UST_ID" "5f9d106a12875025b39777fa" (id 4) (at 95.25 115.57 0)
+      (effects (font (size 1.27 1.27)) hide)
+    )
+  )
