File: hw/sch_pcb/TFPROBE01A.kicad_sch (KiCad schematic)
At the start: 8 parts, among them J1 HEADER_1x03, M3 HOLE, M4 HOLE, U1 AH3572, U2 VCNT2020

Commit message: Update title block.
Other:
- company: (none) -> ThunderFly s.r.o.
- title: (none) -> TFPROBE01A
Changed lines of the file:
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@@
 (kicad_sch (version 20201015) (generator eeschema)
-  (page 1 1)
   (paper "A4")
+  (title_block
+    (title "TFPROBE01A")
+    (date "2021-01-23")
+    (company "ThunderFly s.r.o.")
+    (comment 1 "Omnipolar magnetic and \\n reflective optical probe")
+    (comment 3 "Sensor for \\n TFRPM measuring device")
+  )
   (junction (at 146.05 109.22) (diameter 1.016) (color 0 0 0 0))
   (junction (at 156.21 111.76) (diameter 1.016) (color 0 0 0 0))
