File: hw/sch_pcb/TFPROBE01A.kicad_sch (KiCad schematic)
At the start: 8 parts, among them J1 HEADER_1x03, M3 HOLE, M4 HOLE, U1 AH3572, U2 VCNT2020

Commit message: Edit schema
Parts:
- R2: value - -> 4k7; UST_ID (none) -> 5c70984612875079b91f8995
Changed lines of the file:
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@@
       (effects (font (size 1.27 1.27)) (justify left))
     )
-    (property "Value" "-" (id 1) (at 147.828 104.019 0)
+    (property "Value" "4k7" (id 1) (at 147.828 104.019 0)
       (effects (font (size 1.27 1.27)) (justify left))
     )
@@
     )
     (property "Datasheet" "~" (id 3) (at 146.05 102.87 0)
+      (effects (font (size 1.27 1.27)) hide)
+    )
+    (property "UST_ID" "5c70984612875079b91f8995" (id 4) (at 146.05 102.87 0)
       (effects (font (size 1.27 1.27)) hide)
     )
@@
       (effects (font (size 1.27 1.27)) (justify left bottom) hide)
     )
-    (property "UST_ID" "5f9d106a12875025b39777fa" (id 4) (at 95.25 115.57 0)
+    (property "UST_ID" "5f9d106a12875025b39777fa" (id 6) (at 95.25 115.57 0)
       (effects (font (size 1.27 1.27)) hide)
     )
     (pin "1")
     (pin "2")
+    (pin "3")
     (pin "4")
-    (pin "3")
   )
   (sheet_instances
@@
     )
     (path "/dc0b4ba4-1c58-4194-aa69-1071feb9bfda"
-      (reference "R2") (unit 1) (value "-") (footprint "Mlab_R:SMD-0805")
+      (reference "R2") (unit 1) (value "4k7") (footprint "Mlab_R:SMD-0805")
     )
     (path "/a7f3953c-82c9-48f9-af66-14b131e92525"

Commit message: Changing component values #5
Parts:
- R1: value 180R -> 51R; UST_ID 5c70984512875079b91f8957 -> 5c70984512875079b91f8953
Changed lines of the file:
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@@
       (effects (font (size 1.27 1.27)) (justify left))
     )
-    (property "Value" "180R" (id 1) (at 72.898 102.749 0)
+    (property "Value" "51R" (id 1) (at 72.898 102.749 0)
       (effects (font (size 1.27 1.27)) (justify left))
     )
@@
       (effects (font (size 1.27 1.27)) hide)
     )
-    (property "UST_ID" "5c70984512875079b91f8957" (id 4) (at 71.12 101.6 0)
+    (property "UST_ID" "5c70984512875079b91f8953" (id 4) (at 71.12 101.6 0)
       (effects (font (size 1.27 1.27)) hide)
     )
@@
     )
     (path "/9e12790b-cec9-4dd8-a3af-c20d5c11d549"
-      (reference "R1") (unit 1) (value "180R") (footprint "Mlab_R:SMD-0603")
+      (reference "R1") (unit 1) (value "51R") (footprint "Mlab_R:SMD-0603")
     )
     (path "/dc0b4ba4-1c58-4194-aa69-1071feb9bfda"
