File: hw/sch_pcb/TFPROBE01A.kicad_pcb (KiCad board)
At the start: 2 copper layers, 14 x 10 mm, 8 parts, among them J1 HEADER_1x03, M3 HOLE, M4 HOLE, U1 AH3572, U2 VCNT2020

Commit message: Edit PCB
Other:
- rule pad_to_mask_clearance: 0 -> 0.2
Changed lines of the file:
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@@
-(kicad_pcb (version 20210722) (generator pcbnew)
+(kicad_pcb (version 20211014) (generator pcbnew)
   (general
     (thickness 1.6)
@@
       (dielectric_constraints no)
     )
-    (pad_to_mask_clearance 0)
+    (pad_to_mask_clearance 0.2)
     (pcbplotparams
       (layerselection 0x00012e0_ffffffff)
